File: Hardware/Rele casero.kicad_sch (KiCad schematic)
At the start: 15 parts, among them J1 Screw_Terminal_01x02, J2 Screw_Terminal_01x02, K1 SANYOU_SRD_Form_C, Q1 PN2222A, U1 ESP32C3-SUPERMINI, U2 4N25, U4 SMTS-102

Commit message: Add files via upload
Connections:
- net A0: now also U1.6 (GPIO10); no longer U1.4 (GPIO8)
- net Micro: now also U1.4 (GPIO8)
- no-connect marks 11 -> 12
Changed lines of the file:
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@@
+	)
+	(no_connect
+		(at 50.8 43.18)
+	)
+	(no_connect
+		(at 50.8 33.02)
 	)
 	(no_connect
@@
 	)
 	(no_connect
-		(at 50.8 33.02)
-	)
-	(no_connect
 		(at 22.86 35.56)
 	)
@@
 	(global_label "A0"
 		(shape input)
+		(at 50.8 40.64 0)
+		(fields_autoplaced yes)
+		(effects
+			(font
+				(size 1.27 1.27)
+			)
+			(justify left)
+		)
+		(property "Intersheetrefs" "${INTERSHEET_REFS}"
+			(at 56.0833 40.64 0)
+			(hide yes)
+			(show_name no)
+			(do_not_autoplace no)
+			(effects
+				(font
+					(size 1.27 1.27)
+				)
+				(justify left)
+			)
+		)
+	)
+	(global_label "Micro"
+		(shape input)
 		(at 50.8 35.56 0)
 		(fields_autoplaced yes)
@@
 		)
 		(property "Intersheetrefs" "${INTERSHEET_REFS}"
-			(at 56.0833 35.56 0)
-			(hide yes)
-			(show_name no)
+			(at 58.8652 35.56 0)
+			(hide yes)
+			(show_name no)

Commit message: Add files via upload
Connections:
- net D0: now also U1.6 (GPIO10); no longer U1.5 (GPIO9)
- net GND: now also J1.1 (Pin_1), U3.2 (-VI)
- net VCC: now also U3.1 (+VI), U4.S; no longer D1.1 (K), I2C_OLED1.2 (Pin_2), K1.5, R2.2, TCRT5000.1 (Pin_1), U1.16 (5V), U2.5, U3.3 (+OUT)
- net VBAT: now reaches J1.2 (Pin_2), U4.P
- net 3V3: now reaches U1.14 (3V3)
- net 3V3: now also I2C_OLED1.2 (Pin_2), TCRT5000.1 (Pin_1)
- net A0: no longer names the net of TCRT5000.4 (Pin_4)
- net A0: no longer U1.6 (GPIO10)
- new net 5V: D1.1 (K), K1.5, R2.2, U1.16 (5V), U2.5, U3.3 (+OUT)
- no-connect marks 12 -> 13
Other:
- moved on the sheet: I2C_OLED1, J1, TCRT5000, U3, U4

Commit message: Add files via upload
Parts:
- I2C_OLED1, TCRT5000: footprint Connector_PinSocket_2.00mm:PinSocket_1x04_P2.00mm_Vertical -> Connector_PinSocket_2.54mm:PinSocket_1x04_P2.54mm_Vertical
Connections:
- net Micro: now also U1.8 (GPIO21); no longer U1.4 (GPIO8)
- net SCL: now also U1.3 (GPIO7); no longer U1.9 (GPIO0)
- net SDA: now also U1.4 (GPIO8); no longer U1.8 (GPIO21)
- net at J2.1 (Pin_1): now also K1.1; no longer K1.3
- net at J2.2 (Pin_2): now also K1.3; no longer K1.1
Other:
- moved on the sheet: J2
Changed lines of the file:
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@@
 	)
 	(no_connect
-		(at 50.8 33.02)
-	)
-	(no_connect
 		(at 50.8 30.48)
 	)
@@
 	)
 	(no_connect
+		(at 22.86 45.72)
+	)
+	(no_connect
 		(at 22.86 38.1)
 	)
@@
 	(wire
 		(pts
-			(xy 140.97 45.72) (xy 142.24 45.72)
+			(xy 176.53 38.1) (xy 176.53 41.91)
 		)
 		(stroke
@@
 	(wire
 		(pts
-			(xy 106.68 81.28) (xy 107.95 81.28)
+			(xy 140.97 45.72) (xy 142.24 45.72)
 		)
 		(stroke
@@
 	(wire
 		(pts
-			(xy 158.75 77.47) (xy 161.29 77.47)
+			(xy 106.68 81.28) (xy 107.95 81.28)
 		)
 		(stroke
@@
 	(wire
 		(pts
-			(xy 171.45 22.86) (xy 179.07 22.86)
+			(xy 158.75 77.47) (xy 161.29 77.47)
 		)
 		(stroke
@@
 	(wire
 		(pts
-			(xy 20.32 33.02) (xy 22.86 33.02)
+			(xy 171.45 22.86) (xy 179.07 22.86)
 		)
 		(stroke
@@
 	(wire
 		(pts
-			(xy 142.24 35.56) (xy 142.24 39.37)
+			(xy 20.32 33.02) (xy 22.86 33.02)
 		)
 		(stroke
@@
 	(wire
 		(pts
-			(xy 179.07 22.86) (xy 179.07 30.48)
+			(xy 142.24 35.56) (xy 142.24 39.37)
 		)
 		(stroke
@@
 	(wire
 		(pts
-			(xy 179.07 38.1) (xy 179.07 33.02)
-		)
-		(stroke
-			(width 0)
-			(type default)
-		)
-	)
-	(wire
-		(pts
 			(xy 46.99 74.93) (xy 49.53 74.93)
 		)
@@
 	(wire
 		(pts
-			(xy 62.23 36.83) (xy 66.04 36.83)
+			(xy 63.5 36.83) (xy 66.04 36.83)
 		)
 		(stroke
@@
 	(wire
 		(pts
-			(xy 52.07 45.72) (xy 50.8 45.72)
+			(xy 173.99 40.64) (xy 173.99 41.91)
 		)
 		(stroke
@@
 	(wire
 		(pts
-			(xy 168.91 38.1) (xy 179.07 38.1)
-		)
-		(stroke
-			(width 0)
-			(type default)
-		)
-	)
-	(wire
-		(pts
 			(xy 69.85 69.85) (xy 69.85 74.93)
 		)
@@
 	(wire
 		(pts
-			(xy 62.23 31.75) (xy 62.23 36.83)
+			(xy 63.5 31.75) (xy 63.5 36.83)
 		)
 		(stroke
@@
 	(wire
 		(pts
+			(xy 179.07 40.64) (xy 173.99 40.64)
+		)
+		(stroke
+			(width 0)
+			(type default)
+		)
+	)
+	(wire
+		(pts
 			(xy 16.51 27.94) (xy 22.86 27.94)
 		)
@@
 	(wire
 		(pts
+			(xy 50.8 45.72) (xy 53.34 45.72)
+		)
+		(stroke
+			(width 0)
+			(type default)
+		)
+	)
+	(wire
+		(pts
 			(xy 158.75 38.1) (xy 158.75 39.37)
 		)
@@
 	(wire
 		(pts
-			(xy 21.59 45.72) (xy 22.86 45.72)
+			(xy 148.59 34.29) (xy 148.59 39.37)
 		)
 		(stroke
@@
 	(wire
 		(pts
-			(xy 148.59 34.29) (xy 148.59 39.37)
+			(xy 104.14 35.56) (xy 104.14 46.99)
 		)
 		(stroke
@@
 	(wire
 		(pts
-			(xy 104.14 35.56) (xy 104.14 46.99)
+			(xy 158.75 21.59) (xy 158.75 22.86)
 		)
 		(stroke
@@
 	(wire
 		(pts
-			(xy 158.75 21.59) (xy 158.75 22.86)
+			(xy 179.07 22.86) (xy 179.07 40.64)
 		)
 		(stroke
@@
 	(wire
 		(pts
+			(xy 168.91 38.1) (xy 176.53 38.1)
+		)
+		(stroke
+			(width 0)
+			(type default)
+		)
+	)
+	(wire
+		(pts
 			(xy 46.99 69.85) (xy 46.99 74.93)
 		)
@@
 	(global_label "SCL"
 		(shape input)
-		(at 21.59 45.72 180)
+		(at 50.8 33.02 0)
 		(fields_autoplaced yes)
 		(effects
@@
 				(size 1.27 1.27)
 			)
-			(justify right)
+			(justify left)
 		)
 		(property "Intersheetrefs" "${INTERSHEET_REFS}"
-			(at 15.0972 45.72 0)
+			(at 57.2928 33.02 0)
 			(hide yes)
 			(show_name no)
@@
 					(size 1.27 1.27)
 				)
-				(justify right)
+				(justify left)
 			)
 		)
@@
 	(global_label "Micro"
 		(shape input)
-		(at 62.23 31.75 90)
+		(at 63.5 31.75 90)
 		(fields_autoplaced yes)
 		(effects
@@
 		)
 		(property "Intersheetrefs" "${INTERSHEET_REFS}"
-			(at 62.23 23.6848 90)
+			(at 63.5 23.6848 90)
 			(hide yes)
 			(show_name no)
@@
 	(global_label "SDA"
 		(shape input)
-		(at 52.07 45.72 0)
+		(at 50.8 35.56 0)
 		(fields_autoplaced yes)
 		(effects
@@
 		)
 		(property "Intersheetrefs" "${INTERSHEET_REFS}"
-			(at 58.6233 45.72 0)
+			(at 57.3533 35.56 0)
 			(hide yes)
 			(show_name no)
@@
 	(global_label "Micro"
 		(shape input)
-		(at 50.8 35.56 0)
+		(at 53.34 45.72 0)
 		(fields_autoplaced yes)
 		(effects
@@
 		)
 		(property "Intersheetrefs" "${INTERSHEET_REFS}"
-			(at 58.8652 35.56 0)
+			(at 61.4052 45.72 0)
 			(hide yes)
 			(show_name no)
@@
 	(symbol
 		(lib_id "Connector:Screw_Terminal_01x02")
-		(at 184.15 30.48 0)
+		(at 176.53 46.99 270)
 		(unit 1)
 		(body_style 1)
@@
 		(dnp no)
 		(property "Reference" "J2"
-			(at 186.69 30.4799 0)
+			(at 176.5301 49.53 0)
 			(show_name no)
 			(do_not_autoplace no)
@@
 		)
 		(property "Value" "Screw_Terminal_01x02"
-			(at 165.862 42.672 0)
+			(at 164.338 28.702 0)
 			(show_name no)
 			(do_not_autoplace no)
@@
 		)
 		(property "Footprint" "TerminalBlock_Phoenix:TerminalBlock_Phoenix_MKDS-1,5-2-5.08_1x02_P5.08mm_Horizontal"
-			(at 184.15 30.48 0)
+			(at 176.53 46.99 0)
 			(hide yes)
 			(show_name no)
@@
 		)
 		(property "Datasheet" ""
-			(at 184.15 30.48 0)
+			(at 176.53 46.99 0)
 			(hide yes)
 			(show_name no)
@@
 		)
 		(property "Description" "Generic screw terminal, single row, 01x02, script generated (kicad-library-utils/schlib/autogen/connector/)"
-			(at 184.15 30.48 0)
+			(at 176.53 46.99 0)
 			(hide yes)
 			(show_name no)
@@
 			)
 		)
-		(property "Footprint" "Connector_PinSocket_2.00mm:PinSocket_1x04_P2.00mm_Vertical"
+		(property "Footprint" "Connector_PinSocket_2.54mm:PinSocket_1x04_P2.54mm_Vertical"
 			(at 166.37 74.93 0)
 			(hide yes)
@@
 			)
 		)
-		(property "Footprint" "Connector_PinSocket_2.00mm:PinSocket_1x04_P2.00mm_Vertical"
+		(property "Footprint" "Connector_PinSocket_2.54mm:PinSocket_1x04_P2.54mm_Vertical"
 			(at 113.03 76.2 0)
 			(hide yes)
