File: Hardware/Rele casero.kicad_pcb (KiCad board)
At the start: 2 copper layers, 15 parts, among them J1 Screw_Terminal_01x02, J2 Screw_Terminal_01x02, K1 SANYOU_SRD_Form_C, Q1 PN2222A, U1 ESP32C3-SUPERMINI, U2 4N25, U4 SMTS-102

Commit message: Add files via upload
Parts:
- moved LED1 0.21 mm to (101.5, 104.0)
- moved R2 0.15 mm to (101.5, 106.8)
Connections:
- U1 pad 4: A0 -> Micro
- U1 pad 6: unconnected-(U1-GPIO10-Pad6) -> A0
Routing:
- net VCC: track 254.9 -> 304.5 mm
- net Net-(J2-Pin_2): track 33.9 -> 53.3 mm
- net Micro: track 0.00 -> 17.2 mm
- net SDA: track 0.00 -> 16.4 mm
- net Net-(D1-A): track 55.7 -> 44.6 mm
- net SCL: track 0.00 -> 10.5 mm
- net D0: track 18.5 -> 24.7 mm
- net A0: track 22.1 -> 21.5 mm

Commit message: Add files via upload
Parts:
- moved U4 2.40 mm to (72.5, 79.0)
Connections:
- net Net-(J1-Pin_2) renamed VBAT
- D1 pad 1: VCC -> 5V
- I2C_OLED1 pad 2: VCC -> 3V3
- J1 pad 1: Net-(J1-Pin_1) -> GND
- K1 pad 5: VCC -> 5V
- R2 pad 2: VCC -> 5V
- TCRT5000 pad 1: VCC -> 3V3
- TCRT5000 pad 4: A0 -> unconnected-(TCRT5000-Pin_4-Pad4)
- U1 pad 14: unconnected-(U1-3V3-Pad14) -> 3V3
- U1 pad 16: VCC -> 5V
- U1 pad 5: D0 -> unconnected-(U1-GPIO9-Pad5)
- U1 pad 6: A0 -> D0
- U2 pad 5: VCC -> 5V
- U3 pad 1: Net-(U3-+VI) -> VCC
- U3 pad 2: Net-(J1-Pin_1) -> GND
- U3 pad 3: VCC -> 5V
- U4 pad S: Net-(U3-+VI) -> VCC
Routing:
- net 5V: track 0.00 -> 255.3 mm
- net VCC: track 304.5 -> 60.2 mm
- net Net-(U3-+VI): track 61.3 -> 0.00 mm
- net Net-(J1-Pin_1): track 53.1 -> 0.00 mm
- net 3V3: track 0.00 -> 43.9 mm
- net A0: track 21.5 -> 0.00 mm
- net D0: track 24.7 -> 22.1 mm
- net VBAT: track 6.31 -> 8.22 mm
- net GND: track 0.00 -> 1.21 mm
- net Micro: track 17.2 -> 17.9 mm

Commit message: Add files via upload
Parts:
- I2C_OLED1, TCRT5000: footprint Connector_PinSocket_2.00mm:PinSocket_1x04_P2.00mm_Vertical -> Connector_PinSocket_2.54mm:PinSocket_1x04_P2.54mm_Vertical
- moved J2 18.3 mm to (70.2, 110.2)
- moved K1 9.78 mm to (86.8, 96.8)
- moved TCRT5000 3.06 mm to (116.5, 90.8)
- moved I2C_OLED1 0.50 mm to (116.5, 71.8)
- moved D1 0.28 mm to (105.5, 111.4)
Connections:
- K1 pad 1: Net-(J2-Pin_2) -> Net-(J2-Pin_1)
- K1 pad 3: Net-(J2-Pin_1) -> Net-(J2-Pin_2)
- U1 pad 3: unconnected-(U1-GPIO7-Pad3) -> SCL
- U1 pad 4: Micro -> SDA
- U1 pad 8: SDA -> Micro
- U1 pad 9: SCL -> unconnected-(U1-GPIO0-Pad9)
Routing:
- net Net-(J2-Pin_2): track 53.3 -> 5.73 mm
- net 5V: track 255.3 -> 210.6 mm
- net SCL: track 10.5 -> 29.6 mm
- net Net-(J2-Pin_1): track 24.2 -> 33.8 mm
- net Net-(D1-A): track 44.6 -> 35.1 mm
- net SDA: track 16.4 -> 24.9 mm
- net Micro: track 17.9 -> 9.78 mm
- net D0: track 22.1 -> 14.5 mm
- net GND: track 1.21 -> 0.00 mm
- net 3V3: track 43.9 -> 44.9 mm

Commit message: Add files via upload
Parts:
- moved U4 1.62 mm to (71.1, 78.1)
- moved J1 0.98 mm to (83.2, 77.8)
- moved U2 0.72 mm to (108.7, 109.2)
Routing:
- net 5V: track 210.6 -> 214.6 mm
- net VCC: track 60.6 -> 58.9 mm
- net VBAT: track 8.22 -> 7.46 mm
